Commit message: Add software limits to velocity and position of arm

File: ArmControl/model/MR_arm.urdf (robot description, URDF)
Before this commit: robot mr_arm, 6 links, 5 joints
Joints:
- joint joint_1: limit lower=-1.570796327 upper=1.570796327 effort=10.0 velocity=2.61799 -> lower=-3.141592 upper=3.141592 effort=10.0 velocity=2.61799
