Commit message: fixed rover initial orientation

File: rover_gazebo/urdf/depth_camera.urdf.xacro (robot description, xacro)
@@ -29,15 +29,15 @@
         <gazebo reference="kinect_link">
             <sensor name="camera" type="depth">
-                <update_rate>20</update_rate>
+                <update_rate>1</update_rate>
                 <camera>
                     <horizontal_fov>1.047198</horizontal_fov>
                     <image>
-                        <width>640</width>
-                        <height>480</height>
+                        <width>80</width>
+                        <height>120</height>
                         <format>R8G8B8</format>
                     </image>
                     <clip>
-                        <near>0.05</near>
-                        <far>3</far>
+                        <near>1.05</near>
+                        <far>5</far>
                     </clip>
                 </camera>
@@ -55,6 +55,6 @@
                     <pointCloudTopicName>/camera/depth/points</pointCloudTopicName>
                     <frameName>camera_link</frameName>
-                    <pointCloudCutoff>0.5</pointCloudCutoff>
-                    <pointCloudCutoffMax>3.0</pointCloudCutoffMax>
+                    <pointCloudCutoff>1.05</pointCloudCutoff>
+                    <pointCloudCutoffMax>5.0</pointCloudCutoffMax>
                     <distortionK1>0</distortionK1>
                     <distortionK2>0</distortionK2>

File: rover_gazebo/urdf/rover.urdf.xacro (robot description, xacro)
@@ -13,12 +13,12 @@
             <origin xyz="0 0 0.1" rpy="0 0 0" />
             <geometry>
-                <mesh filename="package://rover_gazebo/meshes/Full_Asm_Adjusted.dae" />
+                <mesh filename="package://rover_gazebo/meshes/rover_body_with_arm.dae" />
             </geometry>
         </visual>
         <collision>
-            <origin xyz="0 0 0.1" rpy="0 0 0" />
+            <origin xyz="0 0 0.4" rpy="0 0 0" />
             <geometry>
                 <!-- <mesh filename="package://rover_gazebo/meshes/Full_Asm_Adjusted.dae"/> -->
-                <box size="0 0 0" />
+                <box size="1 .5 .25" />
             </geometry>
         </collision>
@@ -32,17 +32,17 @@
     </joint>
     <xacro:wheel wheel_prefix="left" parent_link="base_link">
-        <origin xyz="0.5125 -0.316275 ${-0.060752 + .1}" rpy="0 3.141592 0" />
+        <origin xyz="0.316275 0.5125 ${-0.060752 + .1}" rpy="0 3.141592 ${3.141592/2}" />
     </xacro:wheel>
     <xacro:wheel wheel_prefix="right" parent_link="base_link">
-        <origin xyz="-0.5125 -0.316275 ${-0.060752 + .1}" rpy="0 0 0" />
+        <origin xyz="0.316275 -0.5125 ${-0.060752 + .1}" rpy="0 0 ${3.141592/2}" />
     </xacro:wheel>
     <xacro:wheel wheel_prefix="rear_left" parent_link="base_link">
-        <origin xyz="0.5125 0.306875 ${-0.060752 + .1}" rpy="0 3.141592 0" />
+        <origin xyz="-0.306875 0.5125 ${-0.060752 + .1}" rpy="0 3.141592 ${3.141592/2}" />
     </xacro:wheel>
     <xacro:wheel wheel_prefix="rear_right" parent_link="base_link">
-        <origin xyz="-0.5125 0.306875 ${-0.060752 + .1}" rpy="0 0 0" />
+        <origin xyz="-0.306875 -0.5125 ${-0.060752 + .1}" rpy="0 0 ${3.141592/2}" />
     </xacro:wheel>
     <xacro:depth_camera parent_link="base_link">
-        <origin xyz="0 0.2754 ${0.9943 + .1}" rpy="0 0 -1.57079"/>
+        <origin xyz="-0.2754 0 ${0.9943 + .1}" rpy="0 0 0"/>
     </xacro:depth_camera>
     <gazebo>

File: rover_gazebo/urdf/wheel.urdf.xacro (robot description, xacro)
@@ -19,5 +19,5 @@
 				<origin xyz="0 0 0" rpy="${M_PI/2} 0 0" />
 				<geometry>
-					<mesh filename="package://rover_gazebo/meshes/full_wheel_assembly_fixed.dae" />
+					<mesh filename="package://rover_gazebo/meshes/rover_wheel.dae" />
 				</geometry>
 			</visual>

Commit message: Updated rover model. Modified wheels' collision box size. Modified cam position and deleted kinect model.

File: rover_gazebo/urdf/depth_camera.urdf.xacro (robot description, xacro)
@@ -14,5 +14,5 @@
                 </geometry>
             </collision>
-            <visual name="kinect_visual">
+            <!-- <visual name="kinect_visual">
                 <origin xyz="0 0 0" rpy="0 0 0" />
                 <geometry>
@@ -20,5 +20,5 @@
                         scale="1.0 1.0 1.0" />
                 </geometry>
-            </visual>
+            </visual> -->
         </link>
         <joint name="depth_camera_joint" type="fixed">

File: rover_gazebo/urdf/rover.urdf.xacro (robot description, xacro)
@@ -13,5 +13,5 @@
             <origin xyz="0 0 0.1" rpy="0 0 0" />
             <geometry>
-                <mesh filename="package://rover_gazebo/meshes/Full_Asm_Adjusted.dae" />
+                <mesh filename="package://rover_gazebo/meshes/Full_Asm_noarm_mast_cam.dae" />
             </geometry>
         </visual>
@@ -44,5 +44,5 @@
     </xacro:wheel>
     <xacro:depth_camera parent_link="base_link">
-        <origin xyz="0 0.2754 ${0.9943 + .1}" rpy="0 0 -1.57079"/>
+        <origin xyz="0 -0.41 0.32" rpy="0 0 -1.57079"/>
     </xacro:depth_camera>
     <gazebo>

File: rover_gazebo/urdf/wheel.urdf.xacro (robot description, xacro)
@@ -25,5 +25,5 @@
 				<origin xyz="0 0 0" rpy="0 0 ${M_PI/2}" />
 				<geometry>
-					<cylinder length="0.2" radius="0.14" />
+					<cylinder length="0.14" radius="0.147" />
 				</geometry>
 			</collision>
