Commit message: Cleaned up code. Removed unnecessary files

File: rover_gazebo/urdf/rover.urdf.xacro (robot description, xacro)
@@ -2,5 +2,4 @@
 <robot  xmlns:xacro="http://ros.org/wiki/xacro"
         name="rover" >
-    <xacro:include filename="$(find rover_gazebo)/urdf/caster.urdf.xacro" />
     <xacro:include filename="$(find rover_gazebo)/urdf/wheel.urdf.xacro" />
     <xacro:arg name="mesh_enabled" default="false" />
@@ -8,9 +7,9 @@
     <link   name = "base_link">
         <inertial>
-            <origin xyz="-0.108 0 -0.02579" rpy="0 0 0"/>
+            <origin xyz="0 0 0" rpy="0 0 0"/>
             <mass value="3.978"/>
-            <inertia ixx="0.021858680" ixy="0.0" ixz="0.010020353"
-                    iyy="0.078572349" iyz="-0.0"
-                    izz="0.091971324"/>
+            <inertia ixx="0.0282916666667" ixy="0.0" ixz="0.0"
+                    iyy="0.0282916666667" iyz="0.0"
+                    izz="0.05625"/>
         </inertial>
         <visual>
@@ -22,5 +21,5 @@
             </xacro:if>
             <xacro:unless value="$(arg mesh_enabled)">
-                <origin xyz="-0.125 0 -0.01" rpy="0 0 0" />
+                <origin xyz="0 0 -0.01" rpy="0 0 0" />
                 <geometry>
                     <box size="0.25 0.25 0.02" />
@@ -30,5 +29,5 @@
         </visual>
         <collision>
-            <origin xyz="-0.125 0 -0.01" rpy="0 0 0" />
+            <origin xyz="0 0 -0.01" rpy="0 0 0" />
             <geometry>
                 <box size="0.25 0.25 0.02" />
@@ -36,22 +35,22 @@
         </collision>
     </link>
-    <link   name =  "base_footprint"/>
+    <link name = "base_footprint"/>
     <joint name = "base_joint"  type = "fixed">
         <parent link="base_footprint"/>
         <child link="base_link"/>
-        <origin xyz="0.0 0.0 0.09188" rpy="0 0 0" />
+        <origin xyz="0.0 0.0 0.0" rpy="0 0 0" />
         <axis xyz="0 1 0" rpy="0 0 0" />
     </joint>
     <xacro:wheel wheel_prefix="left" parent_link="base_link" >
-        <origin xyz="-0.04 0.14 -0.045" rpy="0 0 0" />
+        <origin xyz="0.14 0.14 -0.045" rpy="0 0 0" />
     </xacro:wheel>
     <xacro:wheel wheel_prefix="right" parent_link="base_link" >
-        <origin xyz="-0.04 -0.14 -0.045" rpy="0 0 0" />
+        <origin xyz="0.14 -0.14 -0.045" rpy="0 0 0" />
     </xacro:wheel>
     <xacro:wheel wheel_prefix="rear_left" parent_link="base_link" >
-        <origin xyz="-0.20 0.14 -0.02533" rpy="0 0 0" />
+        <origin xyz="-0.14 0.14 -0.045" rpy="0 0 0" />
     </xacro:wheel>
     <xacro:wheel wheel_prefix="rear_right" parent_link="base_link" >
-        <origin xyz="-0.20 -0.14 -0.02533" rpy="0 0 0" />
+        <origin xyz="-0.14 -0.14 -0.045" rpy="0 0 0" />
     </xacro:wheel>
     <gazebo>

File: rover_gazebo/urdf/wheel.urdf.xacro (robot description, xacro)
@@ -5,4 +5,5 @@
     <xacro:property name="wheel_mu1" value="10000000" />
     <xacro:property name="wheel_mu2" value="10000000" />
+	<xacro:property name="M_PI" value="3.14159265" />
 <xacro:macro name="wheel" params="wheel_prefix parent_link *joint_pose">
 		<!-- Wheel Link -->
@@ -11,5 +12,5 @@
 				<mass value="0.144" />
 				<origin xyz="0 0 0" />
-				<inertia  ixx="0.00008929863" ixy="0" ixz="0" iyy="0.000168983" iyz="0" izz="0.00008929863" />
+				<inertia  ixx="0.00108333333333" ixy="0" ixz="0" iyy="0.00108333333333" iyz="0" izz="0.002" />
 			</inertial>
 			<visual>
@@ -40,5 +41,5 @@
 			<xacro:insert_block name="joint_pose"/>
 			<axis xyz="0 1 0" rpy="0 0 0" />
-			<dynamics damping="0.5" friction="100.0" />
+			<dynamics damping="1" friction="100.0" />
 		</joint>
 		<gazebo reference="${wheel_prefix}_wheel_link">

Commit message: change mass inertia

File: rover_gazebo/urdf/rover.urdf.xacro (robot description, xacro)
@@ -8,8 +8,8 @@
         <inertial>
             <origin xyz="0 0 0" rpy="0 0 0"/>
-            <mass value="3.978"/>
-            <inertia ixx="0.0282916666667" ixy="0.0" ixz="0.0"
-                    iyy="0.0282916666667" iyz="0.0"
-                    izz="0.05625"/>
+            <mass value="45.2"/>
+            <inertia ixx="1.7724" ixy="0.0" ixz="0.0"
+                    iyy="0.141558" iyz="-0.0"
+                    izz="0.179826"/>
         </inertial>
         <visual>

File: rover_gazebo/urdf/wheel.urdf.xacro (robot description, xacro)
@@ -10,7 +10,7 @@
 		<link name="${wheel_prefix}_wheel_link">
 			<inertial>
-				<mass value="0.144" />
+				<mass value="1.2" />
 				<origin xyz="0 0 0" />
-				<inertia  ixx="0.00108333333333" ixy="0" ixz="0" iyy="0.00108333333333" iyz="0" izz="0.002" />
+				<inertia  ixx="0.142" ixy="0.0003118" ixz="0.0000392177" iyy="0.14155823" iyz="-0.000062645" izz="1.3729" />
 			</inertial>
 			<visual>

Commit message: import meshes

File: rover_gazebo/urdf/rover.urdf.xacro (robot description, xacro)
@@ -14,17 +14,17 @@
         </inertial>
         <visual>
-            <xacro:if value="$(arg mesh_enabled)">
-                <origin xyz="0 0 0" rpy="0 0 0" />
+            <!-- <xacro:if value="$(arg mesh_enabled)"> -->
+                <origin xyz="-0.3 -1.2 -0.3" rpy="1.57 0 1.57" />
                 <geometry>
-                    <mesh filename="package://onebot_description/meshes/base_link.dae" />
+                    <mesh filename="package://rover_gazebo/meshes/2Full_Asm_F2022.dae" scale = "0.001 0.001 0.001"/>
                 </geometry>
-            </xacro:if>
-            <xacro:unless value="$(arg mesh_enabled)">
-                <origin xyz="0 0 -0.01" rpy="0 0 0" />
+            <!-- </xacro:if>
+            <xacro:unless value="$(arg mesh_enabled)"> -->
+                <!-- <origin xyz="0 0 -0.01" rpy="0 0 0" />
                 <geometry>
                     <box size="0.25 0.25 0.02" />
-                </geometry>
-                <material name="Blue" />
-            </xacro:unless>
+                </geometry>  -->
+                <!-- <material name="Blue" />
+            </xacro:unless> -->
         </visual>
         <collision>
@@ -43,5 +43,5 @@
     </joint>
     <xacro:wheel wheel_prefix="left" parent_link="base_link" >
-        <origin xyz="0.14 0.14 -0.045" rpy="0 0 0" />
+        <origin xyz="0.5 0.14 -0.045" rpy="0 0 0" />
     </xacro:wheel>
     <xacro:wheel wheel_prefix="right" parent_link="base_link" >

File: rover_gazebo/urdf/wheel.urdf.xacro (robot description, xacro)
@@ -15,16 +15,11 @@
 			</inertial>
 			<visual>
-				<xacro:if value="$(arg mesh_enabled)">
-					<origin xyz="0 0 0" rpy="0 0 ${M_PI/2}" />
+					<origin xyz="0 0 0" rpy="${M_PI/2} 0 0" />
+					<!-- <geometry>
+						<cylinder length="0.02" radius="0.04688" />
+					</geometry> -->
 					<geometry>
-						<mesh filename="package://rover_gazebo/meshes/wheel.dae" />
+						<mesh filename="package://rover_gazebo/meshes/full wheel assembly v2.dae" scale = "0.001 0.001 0.001"/>
 					</geometry>
-				</xacro:if>
-				<xacro:unless value="$(arg mesh_enabled)">
-					<origin xyz="0 0 0" rpy="${M_PI/2} 0 0" />
-					<geometry>
-						<cylinder length="0.02" radius="0.04688" />
-					</geometry>
-				</xacro:unless>
 			</visual>
 			<collision>

Commit message: Implemented Meshes

File: rover_gazebo/urdf/rover.urdf.xacro (robot description, xacro)
@@ -1,35 +1,23 @@
 <?xml version="1.0"?>
-<robot  xmlns:xacro="http://ros.org/wiki/xacro"
-        name="rover" >
+<robot name="myfirst" xmlns:xacro="http://ros.org/wiki/xacro">
     <xacro:include filename="$(find rover_gazebo)/urdf/wheel.urdf.xacro" />
-    <xacro:arg name="mesh_enabled" default="false" />
-    <xacro:arg name="robot_namespace" default="/"/>
-    <link   name = "base_link">
+    <link name = "base_link">
         <inertial>
             <origin xyz="0 0 0" rpy="0 0 0"/>
             <mass value="45.2"/>
-            <inertia ixx="1.7724" ixy="0.0" ixz="0.0"
-                    iyy="0.141558" iyz="-0.0"
-                    izz="0.179826"/>
+            <!-- <inertia ixx="0" ixy="0.0" ixz="0.0" iyy="0" iyz="0.0" izz="0"/> -->
+            <inertia ixx="1.7724" ixy="0.0" ixz="0.0" iyy="0.141558" iyz="-0.0" izz="0.179826"/>
         </inertial>
         <visual>
-            <!-- <xacro:if value="$(arg mesh_enabled)"> -->
-                <origin xyz="-0.3 -1.2 -0.3" rpy="1.57 0 1.57" />
-                <geometry>
-                    <mesh filename="package://rover_gazebo/meshes/2Full_Asm_F2022.dae" scale = "0.001 0.001 0.001"/>
-                </geometry>
-            <!-- </xacro:if>
-            <xacro:unless value="$(arg mesh_enabled)"> -->
-                <!-- <origin xyz="0 0 -0.01" rpy="0 0 0" />
-                <geometry>
-                    <box size="0.25 0.25 0.02" />
-                </geometry>  -->
-                <!-- <material name="Blue" />
-            </xacro:unless> -->
+            <origin xyz="0 0 0.1" rpy="0 0 0" />
+            <geometry>
+                <mesh filename="package://rover_gazebo/meshes/Full_Asm_Adjusted.dae"/>
+            </geometry>
         </visual>
         <collision>
-            <origin xyz="0 0 -0.01" rpy="0 0 0" />
+            <origin xyz="0 0 0.1" rpy="0 0 0" />
             <geometry>
-                <box size="0.25 0.25 0.02" />
+                <!-- <mesh filename="package://rover_gazebo/meshes/Full_Asm_Adjusted.dae"/> -->
+                <box size="0 0 0" />
             </geometry>
         </collision>
@@ -43,21 +31,19 @@
     </joint>
     <xacro:wheel wheel_prefix="left" parent_link="base_link" >
-        <origin xyz="0.5 0.14 -0.045" rpy="0 0 0" />
+        <origin xyz="0.5125 -0.316275 ${-0.060752 + .1}" rpy="0 3.141592 0" />
     </xacro:wheel>
     <xacro:wheel wheel_prefix="right" parent_link="base_link" >
-        <origin xyz="0.14 -0.14 -0.045" rpy="0 0 0" />
+        <origin xyz="-0.5125 -0.316275 ${-0.060752 + .1}" rpy="0 0 0" />
     </xacro:wheel>
     <xacro:wheel wheel_prefix="rear_left" parent_link="base_link" >
-        <origin xyz="-0.14 0.14 -0.045" rpy="0 0 0" />
+        <origin xyz="0.5125 0.306875 ${-0.060752 + .1}" rpy="0 3.141592 0" />
     </xacro:wheel>
     <xacro:wheel wheel_prefix="rear_right" parent_link="base_link" >
-        <origin xyz="-0.14 -0.14 -0.045" rpy="0 0 0" />
+        <origin xyz="-0.5125 0.306875 ${-0.060752 + .1}" rpy="0 0 0" />
     </xacro:wheel>
     <gazebo>
         <plugin name="gazebo_ros_control" filename="libgazebo_ros_control.so">
-            <robotNamespace>/</robotNamespace>
-        <!-- <robotNamespace>$(arg robot_namespace)</robotNamespace> -->
-        <!-- <legacyModeNS>true</legacyModeNS> -->
+        <robotNamespace>/</robotNamespace>
         </plugin>
-    </gazebo>
+    </gazebo>>
 </robot>

File: rover_gazebo/urdf/wheel.urdf.xacro (robot description, xacro)
@@ -3,6 +3,6 @@
   	<xacro:property name="wheel_kp" value="10000000.0" />
     <xacro:property name="wheel_kd" value="1.0" />
-    <xacro:property name="wheel_mu1" value="200" />
-    <xacro:property name="wheel_mu2" value="100" />
+    <xacro:property name="wheel_mu1" value="5" />
+    <xacro:property name="wheel_mu2" value="5" />
 	<xacro:property name="M_PI" value="3.14159265" />
 <xacro:macro name="wheel" params="wheel_prefix parent_link *joint_pose">
@@ -12,19 +12,17 @@
 				<mass value="1.2" />
 				<origin xyz="0 0 0" />
+				<!-- <inertia  ixx="0" ixy="0" ixz="0" iyy="0" iyz="0" izz="0" /> -->
 				<inertia  ixx="0.142" ixy="0.0003118" ixz="0.0000392177" iyy="0.14155823" iyz="-0.000062645" izz="1.3729" />
 			</inertial>
 			<visual>
-					<origin xyz="0 0 0" rpy="${M_PI/2} 0 0" />
-					<!-- <geometry>
-						<cylinder length="0.02" radius="0.04688" />
-					</geometry> -->
-					<geometry>
-						<mesh filename="package://rover_gazebo/meshes/full wheel assembly v2.dae" scale = "0.001 0.001 0.001"/>
-					</geometry>
+				<origin xyz="0 0 0" rpy="${M_PI/2} 0 0" />
+				<geometry>
+					<mesh filename="package://rover_gazebo/meshes/full_wheel_assembly_fixed.dae"/>
+				</geometry>
 			</visual>
 			<collision>
-				<origin xyz="0 0 0" rpy="${M_PI/2} 0 0" />
+				<origin xyz="0.03 0 0" rpy="0 ${M_PI/2} 0" />
 				<geometry>
-						<cylinder length="0.02" radius="0.04688" />
+						<cylinder length="0.2" radius="0.14" />
 				</geometry>
 			</collision>
@@ -35,6 +33,17 @@
 			<child link="${wheel_prefix}_wheel_link"/>
 			<xacro:insert_block name="joint_pose"/>
-			<axis xyz="0 1 0" rpy="0 0 0" />
-			<limit effort="30" velocity="1.0"/>
+			<xacro:if value="${wheel_prefix == 'left'}">
+				<axis xyz="-1 0 0" rpy="0 0 0" />
+			</xacro:if>
+			<xacro:if value="${wheel_prefix == 'right'}">
+				<axis xyz="1 0 0" rpy="0 0 0" />
+			</xacro:if>
+			<xacro:if value="${wheel_prefix == 'rear_left'}">
+				<axis xyz="-1 0 0" rpy="0 0 0" />
+			</xacro:if>
+			<xacro:if value="${wheel_prefix == 'rear_right'}">
+				<axis xyz="1 0 0" rpy="0 0 0" />
+			</xacro:if>
+			<limit effort="300" velocity="50.0"/>
 			<!-- <dynamics damping="1" friction="100.0" /> -->
 		</joint>

Commit message: Added working depth camera to simulation

File: rover_gazebo/urdf/rover.urdf.xacro (robot description, xacro)
@@ -2,15 +2,16 @@
 <robot name="myfirst" xmlns:xacro="http://ros.org/wiki/xacro">
     <xacro:include filename="$(find rover_gazebo)/urdf/wheel.urdf.xacro" />
-    <link name = "base_link">
+    <xacro:include filename="$(find rover_gazebo)/urdf/depth_camera.urdf.xacro" />
+    <link name="base_link">
         <inertial>
-            <origin xyz="0 0 0" rpy="0 0 0"/>
-            <mass value="45.2"/>
+            <origin xyz="0 0 0" rpy="0 0 0" />
+            <mass value="45.2" />
             <!-- <inertia ixx="0" ixy="0.0" ixz="0.0" iyy="0" iyz="0.0" izz="0"/> -->
-            <inertia ixx="1.7724" ixy="0.0" ixz="0.0" iyy="0.141558" iyz="-0.0" izz="0.179826"/>
+            <inertia ixx="1.7724" ixy="0.0" ixz="0.0" iyy="0.141558" iyz="-0.0" izz="0.179826" />
         </inertial>
         <visual>
             <origin xyz="0 0 0.1" rpy="0 0 0" />
             <geometry>
-                <mesh filename="package://rover_gazebo/meshes/Full_Asm_Adjusted.dae"/>
+                <mesh filename="package://rover_gazebo/meshes/Full_Asm_Adjusted.dae" />
             </geometry>
         </visual>
@@ -23,27 +24,30 @@
         </collision>
     </link>
-    <link name = "base_footprint"/>
-    <joint name = "base_joint"  type = "fixed">
-        <parent link="base_footprint"/>
-        <child link="base_link"/>
+    <link name="base_footprint" />
+    <joint name="base_joint" type="fixed">
+        <parent link="base_footprint" />
+        <child link="base_link" />
         <origin xyz="0.0 0.0 0.0" rpy="0 0 0" />
         <axis xyz="0 1 0" rpy="0 0 0" />
     </joint>
-    <xacro:wheel wheel_prefix="left" parent_link="base_link" >
+    <xacro:wheel wheel_prefix="left" parent_link="base_link">
         <origin xyz="0.5125 -0.316275 ${-0.060752 + .1}" rpy="0 3.141592 0" />
     </xacro:wheel>
-    <xacro:wheel wheel_prefix="right" parent_link="base_link" >
+    <xacro:wheel wheel_prefix="right" parent_link="base_link">
         <origin xyz="-0.5125 -0.316275 ${-0.060752 + .1}" rpy="0 0 0" />
     </xacro:wheel>
-    <xacro:wheel wheel_prefix="rear_left" parent_link="base_link" >
+    <xacro:wheel wheel_prefix="rear_left" parent_link="base_link">
         <origin xyz="0.5125 0.306875 ${-0.060752 + .1}" rpy="0 3.141592 0" />
     </xacro:wheel>
-    <xacro:wheel wheel_prefix="rear_right" parent_link="base_link" >
+    <xacro:wheel wheel_prefix="rear_right" parent_link="base_link">
         <origin xyz="-0.5125 0.306875 ${-0.060752 + .1}" rpy="0 0 0" />
     </xacro:wheel>
+    <xacro:depth_camera parent_link="base_link">
+        <origin xyz="0 0.2754 ${0.9943 + .1}" rpy="0 0 -1.57079"/>
+    </xacro:depth_camera>
     <gazebo>
         <plugin name="gazebo_ros_control" filename="libgazebo_ros_control.so">
-        <robotNamespace>/</robotNamespace>
+            <robotNamespace>/</robotNamespace>
         </plugin>
-    </gazebo>>
+    </gazebo>
 </robot>

File: rover_gazebo/urdf/wheel.urdf.xacro (robot description, xacro)
@@ -1,10 +1,10 @@
 <?xml version="1.0"?>
-<robot name="wheel" xmlns:xacro="http://ros.org/wiki/xacro" >
-  	<xacro:property name="wheel_kp" value="10000000.0" />
-    <xacro:property name="wheel_kd" value="1.0" />
-    <xacro:property name="wheel_mu1" value="5" />
-    <xacro:property name="wheel_mu2" value="5" />
+<robot name="wheel" xmlns:xacro="http://ros.org/wiki/xacro">
+	<xacro:property name="wheel_kp" value="10000000.0" />
+	<xacro:property name="wheel_kd" value="1.0" />
+	<xacro:property name="wheel_mu1" value="5" />
+	<xacro:property name="wheel_mu2" value="5" />
 	<xacro:property name="M_PI" value="3.14159265" />
-<xacro:macro name="wheel" params="wheel_prefix parent_link *joint_pose">
+	<xacro:macro name="wheel" params="wheel_prefix parent_link *joint_pose">
 		<!-- Wheel Link -->
 		<link name="${wheel_prefix}_wheel_link">
@@ -13,10 +13,11 @@
 				<origin xyz="0 0 0" />
 				<!-- <inertia  ixx="0" ixy="0" ixz="0" iyy="0" iyz="0" izz="0" /> -->
-				<inertia  ixx="0.142" ixy="0.0003118" ixz="0.0000392177" iyy="0.14155823" iyz="-0.000062645" izz="1.3729" />
+				<inertia ixx="0.142" ixy="0.0003118" ixz="0.0000392177" iyy="0.14155823"
+					iyz="-0.000062645" izz="1.3729" />
 			</inertial>
 			<visual>
 				<origin xyz="0 0 0" rpy="${M_PI/2} 0 0" />
 				<geometry>
-					<mesh filename="package://rover_gazebo/meshes/full_wheel_assembly_fixed.dae"/>
+					<mesh filename="package://rover_gazebo/meshes/full_wheel_assembly_fixed.dae" />
 				</geometry>
 			</visual>
@@ -24,5 +25,5 @@
 				<origin xyz="0.03 0 0" rpy="0 ${M_PI/2} 0" />
 				<geometry>
-						<cylinder length="0.2" radius="0.14" />
+					<cylinder length="0.2" radius="0.14" />
 				</geometry>
 			</collision>
@@ -30,7 +31,7 @@
 		<!-- Wheel Joint -->
 		<joint name="${wheel_prefix}_wheel" type="continuous">
-			<parent link="${parent_link}"/>
-			<child link="${wheel_prefix}_wheel_link"/>
-			<xacro:insert_block name="joint_pose"/>
+			<parent link="${parent_link}" />
+			<child link="${wheel_prefix}_wheel_link" />
+			<xacro:insert_block name="joint_pose" />
 			<xacro:if value="${wheel_prefix == 'left'}">
 				<axis xyz="-1 0 0" rpy="0 0 0" />
@@ -45,12 +46,12 @@
 				<axis xyz="1 0 0" rpy="0 0 0" />
 			</xacro:if>
-			<limit effort="300" velocity="50.0"/>
+			<limit effort="300" velocity="50.0" />
 			<!-- <dynamics damping="1" friction="100.0" /> -->
 		</joint>
 		<gazebo reference="${wheel_prefix}_wheel_link">
-			<mu1 value="${wheel_mu1}"/>
-			<mu2 value="${wheel_mu2}"/>
-			<kp value ="${wheel_kp}"/>
-    		<kd value ="${wheel_kd}"/>
+			<mu1 value="${wheel_mu1}" />
+			<mu2 value="${wheel_mu2}" />
+			<kp value="${wheel_kp}" />
+			<kd value="${wheel_kd}" />
 			<material>Gazebo/Grey</material>
 		</gazebo>
@@ -64,4 +65,4 @@
 			</joint>
 		</transmission>
-</xacro:macro>
+	</xacro:macro>
 </robot>

Commit message: update urdf

File: rover_gazebo/urdf/rover.urdf.xacro (robot description, xacro)
@@ -1,4 +1,44 @@
 <?xml version="1.0"?>
 <robot name="myfirst" xmlns:xacro="http://ros.org/wiki/xacro">
+    <transmission name="right_transmission">
+        <type>transmission_interface/SimpleTransmission</type>
+        <joint name="right_wheel">
+            <hardwareInterface>hardware_interface/VelocityJointInterface</hardwareInterface>
+        </joint>
+        <actuator name="right_motor">
+            <mechanicalReduction>1.0</mechanicalReduction>
+            <hardwareInterface>hardware_interface/VelocityJointInterface</hardwareInterface>
+        </actuator>
+    </transmission>
+    <transmission name="left_transmission">
+        <type>transmission_interface/SimpleTransmission</type>
+        <joint name="left_wheel">
+            <hardwareInterface>hardware_interface/VelocityJointInterface</hardwareInterface>
+        </joint>
+        <actuator name="left_motor">
+            <mechanicalReduction>1.0</mechanicalReduction>
+            <hardwareInterface>hardware_interface/VelocityJointInterface</hardwareInterface>
+        </actuator>
+    </transmission>
+    <transmission name="rear_right_transmission">
+        <type>transmission_interface/SimpleTransmission</type>
+        <joint name="rear_right_wheel">
+            <hardwareInterface>hardware_interface/VelocityJointInterface</hardwareInterface>
+        </joint>
+        <actuator name="rear_right_motor">
+            <mechanicalReduction>1.0</mechanicalReduction>
+            <hardwareInterface>hardware_interface/VelocityJointInterface</hardwareInterface>
+        </actuator>
+    </transmission>
+    <transmission name="rear_left_transmission">
+        <type>transmission_interface/SimpleTransmission</type>
+        <joint name="rear_left_wheel">
+            <hardwareInterface>hardware_interface/VelocityJointInterface</hardwareInterface>
+        </joint>
+        <actuator name="rear_left_motor">
+            <mechanicalReduction>1.0</mechanicalReduction>
+            <hardwareInterface>hardware_interface/VelocityJointInterface</hardwareInterface>
+        </actuator>
+    </transmission>
     <xacro:include filename="$(find rover_gazebo)/urdf/wheel.urdf.xacro" />
     <xacro:include filename="$(find rover_gazebo)/urdf/depth_camera.urdf.xacro" />
@@ -48,4 +88,5 @@
     <gazebo>
         <plugin name="gazebo_ros_control" filename="libgazebo_ros_control.so">
+            <robotSimType>gazebo_ros_control/DefaultRobotHWSim</robotSimType>
             <robotNamespace>/</robotNamespace>
         </plugin>
