Commit message: Updated the wheels' mesh. Fixed steering on sim.

File: rover_gazebo/urdf/rover.urdf.xacro (robot description, xacro)
@@ -32,14 +32,14 @@
     </joint>
     <xacro:wheel wheel_prefix="left" parent_link="base_link">
-        <origin xyz="0.5125 -0.316275 ${-0.060752 + .1}" rpy="0 3.141592 0" />
+        <origin xyz="0.5125 -0.316275 ${-0.060752 + .1}" rpy="0 1.57079 0" />
     </xacro:wheel>
     <xacro:wheel wheel_prefix="right" parent_link="base_link">
-        <origin xyz="-0.5125 -0.316275 ${-0.060752 + .1}" rpy="0 0 0" />
+        <origin xyz="-0.5125 -0.316275 ${-0.060752 + .1}" rpy="0 1.57079 0" />
     </xacro:wheel>
     <xacro:wheel wheel_prefix="rear_left" parent_link="base_link">
-        <origin xyz="0.5125 0.306875 ${-0.060752 + .1}" rpy="0 3.141592 0" />
+        <origin xyz="0.5125 0.306875 ${-0.060752 + .1}" rpy="0 1.57079 0" />
     </xacro:wheel>
     <xacro:wheel wheel_prefix="rear_right" parent_link="base_link">
-        <origin xyz="-0.5125 0.306875 ${-0.060752 + .1}" rpy="0 0 0" />
+        <origin xyz="-0.5125 0.306875 ${-0.060752 + .1}" rpy="0 1.57079 0" />
     </xacro:wheel>
     <xacro:depth_camera parent_link="base_link">

File: rover_gazebo/urdf/wheel.urdf.xacro (robot description, xacro)
@@ -19,9 +19,9 @@
 				<origin xyz="0 0 0" rpy="${M_PI/2} 0 0" />
 				<geometry>
-					<mesh filename="package://rover_gazebo/meshes/full_wheel_assembly_fixed.dae" />
+					<mesh filename="package://rover_gazebo/meshes/WHEEL.dae" />
 				</geometry>
 			</visual>
 			<collision>
-				<origin xyz="0.03 0 0" rpy="0 ${M_PI/2} 0" />
+				<origin xyz="0 0 0" rpy="0 0 ${M_PI/2}" />
 				<geometry>
 					<cylinder length="0.2" radius="0.14" />
@@ -35,14 +35,14 @@
 			<xacro:insert_block name="joint_pose" />
 			<xacro:if value="${wheel_prefix == 'left'}">
-				<axis xyz="-1 0 0" rpy="0 0 0" />
+				<axis xyz="0 0 1" rpy="0 0 0" />
 			</xacro:if>
 			<xacro:if value="${wheel_prefix == 'right'}">
-				<axis xyz="1 0 0" rpy="0 0 0" />
+				<axis xyz="0 0 1" rpy="0 0 0" />
 			</xacro:if>
 			<xacro:if value="${wheel_prefix == 'rear_left'}">
-				<axis xyz="-1 0 0" rpy="0 0 0" />
+				<axis xyz="0 0 1" rpy="0 0 0" />
 			</xacro:if>
 			<xacro:if value="${wheel_prefix == 'rear_right'}">
-				<axis xyz="1 0 0" rpy="0 0 0" />
+				<axis xyz="0 0 1" rpy="0 0 0" />
 			</xacro:if>
 			<limit effort="300" velocity="50.0" />

Commit message: Created .urdf.xacro arm file Copied arm urdf to rover_gazebo meshes. Modified rover urdf multiple times. Last modification was a trial with the regular urdf (not xacro) arm file. Sim works, but arm is not appearing.

File: rover_gazebo/urdf/rover.urdf.xacro (robot description, xacro)
@@ -3,4 +3,5 @@
     <xacro:include filename="$(find rover_gazebo)/urdf/wheel.urdf.xacro" />
     <xacro:include filename="$(find rover_gazebo)/urdf/depth_camera.urdf.xacro" />
+    <!-- <xacro:include filename="$(find rover_gazebo)/urdf/MR_arm.urdf"/> -->
     <link name="base_link">
         <inertial>
@@ -31,4 +32,9 @@
         <axis xyz="0 1 0" rpy="0 0 0" />
     </joint>
+    <joint name="arm_joint" type="fixed">
+        <parent link="base_footprint"/>
+        <child link="link_0"/>
+        <origin xyz="0 1 0" rpy="0 0 0"/>
+    </joint>
     <xacro:wheel wheel_prefix="left" parent_link="base_link">
         <origin xyz="0.5125 -0.316275 ${-0.060752 + .1}" rpy="0 1.57079 0" />
@@ -46,4 +52,5 @@
         <origin xyz="0 -0.41 0.32" rpy="0 0 -1.57079"/>
     </xacro:depth_camera>
+   <xacro:include filename="$(find rover_gazebo)/urdf/MR_arm.urdf"/>
     <gazebo>
         <plugin name="gazebo_ros_control" filename="libgazebo_ros_control.so">

Commit message: added mars map to mcgillrover. added wheel odometry and IMU fusion. added a single launch file (combined.launch to launch everything).

File: rover_gazebo/urdf/rover.urdf.xacro (robot description, xacro)
@@ -1,4 +1,5 @@
 <?xml version="1.0"?>
 <robot name="myfirst" xmlns:xacro="http://ros.org/wiki/xacro">
+    <!-- Include other URDF files -->
     <xacro:include filename="$(find rover_gazebo)/urdf/wheel.urdf.xacro" />
     <xacro:include filename="$(find rover_gazebo)/urdf/depth_camera.urdf.xacro" />
@@ -7,5 +8,4 @@
             <origin xyz="0 0 0" rpy="0 0 0" />
             <mass value="45.2" />
-            <!-- <inertia ixx="0" ixy="0.0" ixz="0.0" iyy="0" iyz="0.0" izz="0"/> -->
             <inertia ixx="1.7724" ixy="0.0" ixz="0.0" iyy="0.141558" iyz="-0.0" izz="0.179826" />
         </inertial>
@@ -19,5 +19,4 @@
             <origin xyz="0 0 0.4" rpy="0 0 0" />
             <geometry>
-                <!-- <mesh filename="package://rover_gazebo/meshes/Full_Asm_Adjusted.dae"/> -->
                 <box size="1 .5 .25" />
             </geometry>
@@ -29,6 +28,6 @@
         <child link="base_link" />
         <origin xyz="0.0 0.0 0.0" rpy="0 0 0" />
-        <axis xyz="0 1 0" rpy="0 0 0" />
     </joint>
+    <!-- Wheels -->
     <xacro:wheel wheel_prefix="left" parent_link="base_link">
         <origin xyz="0.316275 0.5125 ${-0.060752 + .1}" rpy="0 3.141592 ${3.141592/2}" />
@@ -43,11 +42,52 @@
         <origin xyz="-0.306875 -0.5125 ${-0.060752 + .1}" rpy="0 0 ${3.141592/2}" />
     </xacro:wheel>
+    <!-- Depth Camera -->
     <xacro:depth_camera parent_link="base_link">
-        <origin xyz="-0.2754 0 ${0.9943 + .1}" rpy="0 0 0"/>
+        <origin xyz="-0.2754 0 ${0.9943 + .1}" rpy="0 0 0" />
     </xacro:depth_camera>
+    <!-- IMU sensor -->
+    <joint name="imu_joint" type="fixed">
+        <axis xyz="1 0 0"/>
+        <origin xyz="0 0 0.205"/>  <!-- Raised 10 cm higher -->
+        <parent link="base_link"/>
+        <child link="imu_link"/>
+    </joint>
+    <link name="imu_link">
+        <inertial>
+            <mass value="0.001"/>
+            <origin rpy="0 0 0" xyz="0 0 0"/>
+            <inertia ixx="0.0001" ixy="0" ixz="0" iyy="0.000001" iyz="0" izz="0.0001"/>
+        </inertial>
+        <visual>
+            <origin rpy="0 0 0" xyz="0 0 0"/>
+            <geometry>
+                <box size="0.05 0.05 0.05"/>  <!-- Smaller size -->
+            </geometry>
+            <!-- Red material definition -->
+            <material name="red">
+                <color rgba="1.0 0.0 0.0 1.0"/>
+            </material>
+        </visual>
+        <collision>
+            <origin rpy="0 0 0" xyz="0 0 0"/>
+            <geometry>
+                <box size="0.05 0.05 0.05"/>  <!-- Smaller size -->
+            </geometry>
+        </collision>
+    </link>
     <gazebo>
         <plugin name="gazebo_ros_control" filename="libgazebo_ros_control.so">
             <robotNamespace>/</robotNamespace>
         </plugin>
+        <!-- IMU Sensor Plugin for Gazebo -->
+        <plugin name="imu_sensor_plugin" filename="libgazebo_ros_imu.so">
+            <alwaysOn>true</alwaysOn>
+            <updateRate>50.0</updateRate>
+            <bodyName>imu_link</bodyName>
+            <topicName>/imu/data</topicName>
+            <gaussianNoise>2.89e-08</gaussianNoise>
+            <xyzOffsets>0 0 0</xyzOffsets>
+            <rpyOffsets>0 0 0</rpyOffsets>
+        </plugin>
     </gazebo>
 </robot>

File: rover_gazebo/worlds/marsyard2022.world.xacro (robot description, xacro)
@@ -32,27 +32,5 @@
       <uri>model://marsyard2022_terrain</uri>
     </include>
-    <xacro:include filename="sdf/landmark.sdf.xacro" />
-    <xacro:macro name="landmark_with_offset" params="id x y z yaw">
-      <xacro:property name="x_offset" value="-17.003807" />
-      <xacro:property name="y_offset" value="7.617856" />
-      <xacro:property name="z_offset" value="1.352268" />
-      <xacro:landmark id="${id}">
-        <pose>${x + x_offset} ${y + y_offset} ${z + z_offset} 0 0 ${yaw}</pose>
-      </xacro:landmark>
-    </xacro:macro>
-    <xacro:landmark_with_offset id="1" x="10.0" y="0.0" z="-0.18" yaw="0.0" />
-    <xacro:landmark_with_offset id="2" x="10.0" y="-10.0" z="-0.46" yaw="0.0" />
-    <xacro:landmark_with_offset id="3" x="28.35" y="-0.04" z="-0.09" yaw="-0.50" />
-    <xacro:landmark_with_offset id="4" x="21.83" y="-2.80" z="-0.28" yaw="-0.29" />
-    <xacro:landmark_with_offset id="5" x="18.71" y="-17.19" z="0.23" yaw="0.53" />
-    <xacro:landmark_with_offset id="6" x="26.95" y="-7.44" z="-0.08" yaw="-1.35" />
-    <xacro:landmark_with_offset id="7" x="15.97" y="7.57" z="-0.41" yaw="-1.31" />
-    <xacro:landmark_with_offset id="8" x="17.87" y="-7.57" z="0.10" yaw="-0.79" />
-    <xacro:landmark_with_offset id="9" x="10.0" y="10.0" z="-0.39" yaw="-0.90" />
-    <xacro:landmark_with_offset id="10" x="29.26" y="-14.52" z="0.13" yaw="-1.52" />
-    <xacro:landmark_with_offset id="11" x="18.41" y="-25.83" z="0.31" yaw="0.08" />
-    <xacro:landmark_with_offset id="12" x="23.34" y="-14.11" z="0.63" yaw="-0.10" />
-    <xacro:landmark_with_offset id="13" x="8.18" y="-18.63" z="0.44" yaw="-0.40" />
-    <xacro:landmark_with_offset id="15" x="2.27" y="-16.84" z="-0.1" yaw="-0.56" />
+    <!-- Removed the landmarks section as it was not needed -->
   </world>
 </sdf>
