Commit message: Added arm to the sim.

File: arm_control/model/MR_arm.urdf.xacro (robot description, xacro)
@@ -9,18 +9,23 @@
 		</joint>
     <link name="link_0">
-      <visual>
-        <origin xyz="0 0 0" rpy="0 0 0" />
-        <geometry>
-          <mesh filename="package://arm_control/meshes/Link0.stl" />
-        </geometry>
-      </visual>
-      <collision>
-        <origin xyz="0 0 0" rpy="0 0 0" />
-        <geometry>
-          <mesh filename="package://arm_control/meshes/collision_Link0.stl" />
-        </geometry>
-      </collision>
-    </link>
-    <joint name="joint_1" type="revolute">
+      <inertial>
+          <mass value="0.1" />
+          <origin xyz="0 0 0" rpy="0 0 0" />
+          <inertia ixx="0" ixy="0" ixz="0" iyy="0" iyz="0" izz="0" />
+      </inertial>
+      <visual>
+        <origin xyz="0 0 0" rpy="0 0 0" />
+        <geometry>
+          <mesh filename="package://arm_control/model/meshes/Link0.stl" />
+        </geometry>
+      </visual>
+      <collision>
+        <origin xyz="0 0 0" rpy="0 0 0" />
+        <geometry>
+          <mesh filename="package://arm_control/model/meshes/collision_Link0.stl" />
+        </geometry>
+      </collision>
+    </link>
+    <joint name="joint_1" type="fixed">
       <origin xyz="0 0 0" rpy="0 0 0" />
       <parent link="link_0" />
@@ -32,14 +37,19 @@
     <!-- Joint 1 -->
     <link name="link_1">
-      <visual>
-        <origin xyz="0 0 0" rpy="0 0 0" />
-        <geometry>
-          <mesh filename="package://arm_control/meshes/Link1.stl" />
-        </geometry>
-      </visual>
-      <collision>
-        <origin xyz="0 0 0" rpy="0 0 0" />
-        <geometry>
-          <mesh filename="package://arm_control/meshes/collision_Link1.stl" />
+      <inertial>
+          <mass value="0.1" />
+          <origin xyz="0 0 0" rpy="0 0 0" />
+          <inertia ixx="0" ixy="0" ixz="0" iyy="0" iyz="0" izz="0" />
+      </inertial>
+      <visual>
+        <origin xyz="0 0 0" rpy="0 0 0" />
+        <geometry>
+          <mesh filename="package://arm_control/model/meshes/Link1.stl" />
+        </geometry>
+      </visual>
+      <collision>
+        <origin xyz="0 0 0" rpy="0 0 0" />
+        <geometry>
+          <mesh filename="package://arm_control/model/meshes/collision_Link1.stl" />
         </geometry>
       </collision>
@@ -54,14 +64,19 @@
     </joint>
     <link name="link_2">
-      <visual>
-        <origin xyz="0 0 0" rpy="0 0 0" />
-        <geometry>
-          <mesh filename="package://arm_control/meshes/Link2.stl" />
-        </geometry>
-      </visual>
-      <collision>
-        <origin xyz="0 0 0" rpy="0 0 0" />
-        <geometry>
-          <mesh filename="package://arm_control/meshes/collision_Link2.stl" />
+      <inertial>
+          <mass value="0.1" />
+          <origin xyz="0 0 0" rpy="0 0 0" />
+          <inertia ixx="0" ixy="0" ixz="0" iyy="0" iyz="0" izz="0" />
+      </inertial>
+      <visual>
+        <origin xyz="0 0 0" rpy="0 0 0" />
+        <geometry>
+          <mesh filename="package://arm_control/model/meshes/Link2.stl" />
+        </geometry>
+      </visual>
+      <collision>
+        <origin xyz="0 0 0" rpy="0 0 0" />
+        <geometry>
+          <mesh filename="package://arm_control/model/meshes/collision_Link2.stl" />
         </geometry>
       </collision>
@@ -76,14 +91,19 @@
     </joint>
     <link name="link_3">
-      <visual>
-        <origin xyz="0 0 0" rpy="0 0 0" />
-        <geometry>
-          <mesh filename="package://arm_control/meshes/Link3.stl" />
-        </geometry>
-      </visual>
-      <collision>
-        <origin xyz="0 0 0" rpy="0 0 0" />
-        <geometry>
-          <mesh filename="package://arm_control/meshes/collision_Link3.stl" />
+      <inertial>
+          <mass value="0.1" />
+          <origin xyz="0 0 0" rpy="0 0 0" />
+          <inertia ixx="0" ixy="0" ixz="0" iyy="0" iyz="0" izz="0" />
+      </inertial>
+      <visual>
+        <origin xyz="0 0 0" rpy="0 0 0" />
+        <geometry>
+          <mesh filename="package://arm_control/model/meshes/Link3.stl" />
+        </geometry>
+      </visual>
+      <collision>
+        <origin xyz="0 0 0" rpy="0 0 0" />
+        <geometry>
+          <mesh filename="package://arm_control/model/meshes/collision_Link3.stl" />
         </geometry>
       </collision>
@@ -98,14 +118,19 @@
     </joint>
     <link name="link_4">
-      <visual>
-        <origin xyz="0 0 0" rpy="0 0 0" />
-        <geometry>
-          <mesh filename="package://arm_control/meshes/Link4.stl" />
-        </geometry>
-      </visual>
-      <collision>
-        <origin xyz="0 0 0" rpy="0 0 0" />
-        <geometry>
-          <mesh filename="package://arm_control/meshes/collision_Link4.stl" />
+      <inertial>
+          <mass value="0.1" />
+          <origin xyz="0 0 0" rpy="0 0 0" />
+          <inertia ixx="0" ixy="0" ixz="0" iyy="0" iyz="0" izz="0" />
+      </inertial>
+      <visual>
+        <origin xyz="0 0 0" rpy="0 0 0" />
+        <geometry>
+          <mesh filename="package://arm_control/model/meshes/Link4.stl" />
+        </geometry>
+      </visual>
+      <collision>
+        <origin xyz="0 0 0" rpy="0 0 0" />
+        <geometry>
+          <mesh filename="package://arm_control/model/meshes/collision_Link4.stl" />
         </geometry>
       </collision>
@@ -120,14 +145,19 @@
     </joint>
     <link name="link_5">
-      <visual>
-        <origin xyz="0 0 0" rpy="0 0 0" />
-        <geometry>
-          <mesh filename="package://arm_control/meshes/Link5.stl" />
-        </geometry>
-      </visual>
-      <collision>
-        <origin xyz="0 0 0" rpy="0 0 0" />
-        <geometry>
-          <mesh filename="package://arm_control/meshes/collision_Link5.stl" />
+      <inertial>
+          <mass value="0.1" />
+          <origin xyz="0 0 0" rpy="0 0 0" />
+          <inertia ixx="0" ixy="0" ixz="0" iyy="0" iyz="0" izz="0" />
+      </inertial>
+      <visual>
+        <origin xyz="0 0 0" rpy="0 0 0" />
+        <geometry>
+          <mesh filename="package://arm_control/model/meshes/Link5.stl" />
+        </geometry>
+      </visual>
+      <collision>
+        <origin xyz="0 0 0" rpy="0 0 0" />
+        <geometry>
+          <mesh filename="package://arm_control/model/meshes/collision_Link5.stl" />
         </geometry>
       </collision>
@@ -150,4 +180,9 @@
     </joint>
     <link name="link_6">
+      <inertial>
+          <mass value="0.1" />
+          <origin xyz="0 0 0" rpy="0 0 0" />
+          <inertia ixx="0" ixy="0" ixz="0" iyy="0" iyz="0" izz="0" />
+      </inertial>
       <visual>
         <origin xyz="0 0 0" rpy="0 0 0" />
@@ -164,4 +199,9 @@
     </link>
     <link name="link_7">
+      <inertial>
+          <mass value="0.1" />
+          <origin xyz="0 0 0" rpy="0 0 0" />
+          <inertia ixx="0" ixy="0" ixz="0" iyy="0" iyz="0" izz="0" />
+      </inertial>
       <visual>
         <origin xyz="0 0 0" rpy="0 0 0" />

File: rover_gazebo/urdf/rover.urdf.xacro (robot description, xacro)
@@ -3,5 +3,5 @@
     <xacro:include filename="$(find rover_gazebo)/urdf/wheel.urdf.xacro" />
     <xacro:include filename="$(find rover_gazebo)/urdf/depth_camera.urdf.xacro" />
-    <!-- <xacro:include filename="$(find rover_gazebo)/urdf/MR_arm.urdf"/> -->
+    <xacro:include filename="$(find arm_control)/model/MR_arm.urdf.xacro"/>
     <link name="base_link">
         <inertial>
@@ -32,9 +32,4 @@
         <axis xyz="0 1 0" rpy="0 0 0" />
     </joint>
-    <joint name="arm_joint" type="fixed">
-        <parent link="base_footprint"/>
-        <child link="link_0"/>
-        <origin xyz="0 1 0" rpy="0 0 0"/>
-    </joint>
     <xacro:wheel wheel_prefix="left" parent_link="base_link">
         <origin xyz="0.5125 -0.316275 ${-0.060752 + .1}" rpy="0 1.57079 0" />
@@ -52,5 +47,7 @@
         <origin xyz="0 -0.41 0.32" rpy="0 0 -1.57079"/>
     </xacro:depth_camera>
-   <xacro:include filename="$(find rover_gazebo)/urdf/MR_arm.urdf"/>
+   <xacro:MR_arm parent_link="base_link">
+        <origin xyz="0 -0.28 0.37" rpy="0 0 -1.57079"/>
+    </xacro:MR_arm>
     <gazebo>
         <plugin name="gazebo_ros_control" filename="libgazebo_ros_control.so">

Commit message: Added transmissions to each joint. Declared position controllers for each joint. Added controllers to Rover launch file.

File: arm_control/model/MR_arm.urdf.xacro (robot description, xacro)
@@ -3,5 +3,5 @@
   <xacro:macro name="MR_arm" params="parent_link *joint_pose">
     <!-- Base link is the center of the robot's bottom plate -->
-    <joint name="MR_arm_joint" type="continuous">
+    <joint name="MR_arm_joint" type="fixed">
 			<parent link="${parent_link}" />
 			<child link="link_0" />
@@ -27,5 +27,5 @@
       </collision>
     </link>
-    <joint name="joint_1" type="fixed">
+    <joint name="joint_1" type="continuous">
       <origin xyz="0 0 0" rpy="0 0 0" />
       <parent link="link_0" />
@@ -217,4 +217,67 @@
       </collision>
     </link>
+    <transmission name="joint_1_trans">
+			<type>transmission_interface/SimpleTransmission</type>
+			<actuator name="joint_1_motor">
+				<mechanicalReduction>1</mechanicalReduction>
+			</actuator>
+			<joint name="joint_1">
+				<hardwareInterface>hardware_interface/PositionJointInterface</hardwareInterface>
+			</joint>
+		</transmission>
+    <transmission name="joint_2_trans">
+			<type>transmission_interface/SimpleTransmission</type>
+			<actuator name="joint_2_motor">
+				<mechanicalReduction>1</mechanicalReduction>
+			</actuator>
+			<joint name="joint_2">
+				<hardwareInterface>hardware_interface/PositionJointInterface</hardwareInterface>
+			</joint>
+		</transmission>
+    <transmission name="joint_3_trans">
+			<type>transmission_interface/SimpleTransmission</type>
+			<actuator name="joint_3_motor">
+				<mechanicalReduction>1</mechanicalReduction>
+			</actuator>
+			<joint name="joint_3">
+				<hardwareInterface>hardware_interface/PositionJointInterface</hardwareInterface>
+			</joint>
+		</transmission>
+        <transmission name="joint_4_trans">
+			<type>transmission_interface/SimpleTransmission</type>
+			<actuator name="joint_4_motor">
+				<mechanicalReduction>1</mechanicalReduction>
+			</actuator>
+			<joint name="joint_4">
+				<hardwareInterface>hardware_interface/PositionJointInterface</hardwareInterface>
+			</joint>
+		</transmission>
+    <transmission name="joint_5_trans">
+			<type>transmission_interface/SimpleTransmission</type>
+			<actuator name="joint_5_motor">
+				<mechanicalReduction>1</mechanicalReduction>
+			</actuator>
+			<joint name="joint_5">
+				<hardwareInterface>hardware_interface/PositionJointInterface</hardwareInterface>
+			</joint>
+		</transmission>
+    <transmission name="joint_6_trans">
+			<type>transmission_interface/SimpleTransmission</type>
+			<actuator name="joint_6_motor">
+				<mechanicalReduction>1</mechanicalReduction>
+			</actuator>
+			<joint name="joint_6">
+				<hardwareInterface>hardware_interface/PositionJointInterface</hardwareInterface>
+			</joint>
+		</transmission>
+    <transmission name="joint_7_trans">
+			<type>transmission_interface/SimpleTransmission</type>
+			<actuator name="joint_7_motor">
+				<mechanicalReduction>1</mechanicalReduction>
+			</actuator>
+			<joint name="joint_7">
+				<hardwareInterface>hardware_interface/PositionJointInterface</hardwareInterface>
+			</joint>
+		</transmission>
   </xacro:macro>
 </robot>

Commit message: Updated transmission types and controller types.

File: arm_control/model/MR_arm.urdf.xacro (robot description, xacro)
@@ -188,5 +188,5 @@
         <origin xyz="0 0 0" rpy="0 0 0" />
         <geometry>
-          <mesh filename="package://arm_control/meshes/finger.stl" />
+          <mesh filename="package://arm_control/model/meshes/finger.stl" />
         </geometry>
       </visual>
@@ -207,5 +207,5 @@
         <origin xyz="0 0 0" rpy="0 0 0" />
         <geometry>
-          <mesh filename="package://arm_control/meshes/finger.stl" />
+          <mesh filename="package://arm_control/model/meshes/finger.stl" />
         </geometry>
       </visual>
