Commit message: added claw model

File: arm_control/model/MR_arm.urdf (robot description, URDF)
Before this commit: robot mr_arm, 6 links, 5 joints
Links:
- added link link_6; collision box size=0.1 0.1 0.1; visual mesh filename=meshes/finger.stl
- added link link_7; collision box size=0.1 0.1 0.1; visual mesh filename=meshes/finger.stl
Joints:
- added joint joint_6: type revolute, parent link_5, child link_6, origin xyz=0.050 -0.045 -0.01 rpy=0 0 1.570796327, axis 0 0 1, limit lower=-3.141592 upper=3.141592 effort=10.0 velocity=2.61799
- added joint joint_7: type revolute, parent link_5, child link_7, origin xyz=0.050 0.045 -0.01 rpy=0 3.141592 1.570796327, axis 0 0 1, limit lower=-3.141592 upper=3.141592 effort=10.0 velocity=2.61799

Commit message: added arm viz

File: arm_control/model/MR_arm.urdf (robot description, URDF)
Before this commit: robot mr_arm, 8 links, 7 joints
Links:
- link link_0: geometry collision mesh filename=package://arm_control/model/meshes/collision_Link0.stl; visual mesh filename=package://arm_control/model/meshes/Link0.stl
- link link_1: geometry collision mesh filename=package://arm_control/model/meshes/collision_Link1.stl; visual mesh filename=package://arm_control/model/meshes/Link1.stl
- link link_2: geometry collision mesh filename=package://arm_control/model/meshes/collision_Link2.stl; visual mesh filename=package://arm_control/model/meshes/Link2.stl
- link link_3: geometry collision mesh filename=package://arm_control/model/meshes/collision_Link3.stl; visual mesh filename=package://arm_control/model/meshes/Link3.stl
- link link_4: geometry collision mesh filename=package://arm_control/model/meshes/collision_Link4.stl; visual mesh filename=package://arm_control/model/meshes/Link4.stl
- link link_5: geometry collision mesh filename=package://arm_control/model/meshes/collision_Link5.stl; visual mesh filename=package://arm_control/model/meshes/Link5.stl
- link link_6: geometry collision box size=0.1 0.1 0.1; visual mesh filename=package://arm_control/model/meshes/finger.stl
- link link_7: geometry collision box size=0.1 0.1 0.1; visual mesh filename=package://arm_control/model/meshes/finger.stl

Commit message: fixup! joystick update

File: arm_control/model/MR_arm.urdf (robot description, URDF)
Before this commit: robot mr_arm, 8 links, 7 joints
Joints:
- removed joint joint_1
- removed joint joint_2
- removed joint joint_3
- removed joint joint_4
- removed joint joint_5
- removed joint joint_6
- added joint joint_elbow: type revolute, parent link_2, child link_3, origin xyz=0 0 0.5 rpy=0 0 0, axis 0 1 0, limit lower=-1.570796327 upper=1.570796327 effort=10.0 velocity=2.61799
- added joint joint_end_effector: type revolute, parent link_5, child link_6, origin xyz=0.050 -0.045 -0.01 rpy=0 0 1.570796327, axis 0 0 1, limit lower=-3.141592 upper=3.141592 effort=10.0 velocity=2.61799
- added joint joint_shoulder: type revolute, parent link_1, child link_2, origin xyz=0 0 0.0575 rpy=0 0 0, axis 0 1 0, limit lower=-1.570796327 upper=1.570796327 effort=10.0 velocity=2.61799
- added joint joint_waist: type revolute, parent link_0, child link_1, origin xyz=0 0 0 rpy=0 0 0, axis 0 0 1, limit lower=-3.141592 upper=3.141592 effort=10.0 velocity=2.61799
- added joint joint_wrist_pitch: type revolute, parent link_3, child link_4, origin xyz=0.4 0 0 rpy=0 0 0, axis 0 1 0, limit lower=-1.570796327 upper=1.570796327 effort=10.0 velocity=2.61799
- added joint joint_wrist_roll: type revolute, parent link_4, child link_5, origin xyz=0.034 0 0 rpy=0 0 0, axis 1 0 0, limit lower=-3.141592 upper=3.141592 effort=10.0 velocity=2.61799

Commit message: Squashed commit of the following:
commit 0d56d5a2b1dd9f7c6a1963beaa9321b075eaddc5
Author: Your Name <you@example.com>
Date:   Fri Jul 26 18:29:30 2024 -0700

    double rviz arm WIP

commit e4c0d74632ede332224419cd963e40ce7f3b3ccb
Author: Your Name <you@example.com>
Date:   Thu Jul 25 21:23:26 2024 -0700

    fixup! joystick update

commit 4af4ed6b7faf71f2b9a4556cad64efd2f4d04f85
Author: mn297 <Peterwayne3293@gmail.com>
Date:   Wed Jul 24 22:34:29 2024 -0400

    fixup! cleanup odrive logic

commit 594c88182c1cdf25f6061ec8dbeb22ea81b892e0
Author: mn297 <Peterwayne3293@gmail.com>
Date:   Sun Jul 21 00:15:07 2024 -0400

    cleanup odrive logic

commit 704314958149dc132d2260abf482d4207c8d412b
Author: mn297 <Peterwayne3293@gmail.com>
Date:   Sat Jul 20 22:18:34 2024 -0400

    refactor drive code

commit 1f572d50a48e370bec128e4ff440a3b296596772
Author: mn297 <peterwayne3293@gmail.com>
Date:   Sat Jul 20 12:00:54 2024 -0400

    joystick update

commit 7b6284bb53e8ea25c33dcdb9c87c407e757e178b
Author: mn297 <peterwayne3293@gmail.com>
Date:   Fri Jul 19 19:48:57 2024 -0400

    added arm viz

commit b7251dca7f028c1125b107dcc775ebbcd191b5c7
Author: Your Name <peterwayne3293@gmail.com>
Date:   Mon Mar 11 18:17:31 2024 -0400

    formatter arm_control

commit 5ccb2dc80625238264f1b1609f17b6acc934d443
Author: mn297 <peterwayne3293@gmail.com>
Date:   Mon Jul 15 19:44:54 2024 -0400

    cleanup GUI code

commit 6d0fc4735b28a93f210288250df2f4e505a22e84
Author: mn297 <peterwayne3293@gmail.com>
Date:   Sun Jul 7 23:07:50 2024 -0400

    refactored structure

commit 95a24dae18dcdc637ea066ef106a2fce9824869d
Author: mn297 <Peterwayne3293@gmail.com>
Date:   Sat Jun 29 21:59:18 2024 -0400

    added limits variable for arm

commit 1216fc379c5bf81e2862f394a9ac692ac583ddc8
Author: mn297 <Peterwayne3293@gmail.com>
Date:   Thu Jun 27 19:16:11 2024 -0400

    cleaning up odrive logic

commit c73ee0e553b3eff64dea19183899912c623faf81
Author: mn297 <Peterwayne3293@gmail.com>
Date:   Thu Jun 27 19:15:09 2024 -0400

    changed brushed to manual

commit cecea7008c94747e61c45d110cf9fcfc4e9a32dd
Author: mn297 <Peterwayne3293@gmail.com>
Date:   Fri Apr 5 21:57:18 2024 -0400

    updated GUI with odrive brushless fb

commit 3267755883f4e3136801eebb3485a703023eb51b
Author: mn297 <Peterwayne3293@gmail.com>
Date:   Fri Apr 5 18:15:17 2024 -0400

    updated arm config

commit 9a2b9a8f373d31da2bd16902d328eb2059ff391c
Author: mn297 <Peterwayne3293@gmail.com>
Date:   Thu Apr 4 22:15:01 2024 -0400

    trim dead code

commit 73085fddc6f6a4610cb37b2472061c375d44c2c9
Author: mn297 <Peterwayne3293@gmail.com>
Date:   Thu Apr 4 19:44:40 2024 -0400

    debugging arm

commit bd33561092a723b7472bd8047663f15d23b38f72
Author: mn297 <Peterwayne3293@gmail.com>
Date:   Thu Apr 4 17:19:02 2024 -0400

    fully resilient with new reconnection logic

commit c52d3f584cff0167949eff869b9a8fed9ad66822
Author: Your Name <peterwayne3293@gmail.com>
Date:   Wed Apr 3 14:11:57 2024 -0400

    big reconnection logic refactor to better OOP patterns

commit 62064227da7c10f4eb838f87c2c467f01701a1a4
Author: Your Name <peterwayne3293@gmail.com>
Date:   Wed Apr 3 00:09:19 2024 -0400

    refactored reconnection logic

commit aa6d36c08b5fcdb35f39eb158cfc13a1cacd94c6
Author: Your Name <peterwayne3293@gmail.com>
Date:   Tue Apr 2 23:28:54 2024 -0400

    odrive status msg change

commit ac6c06e5a5f5e21661a79296c88ad32396d4bde5
Author: mn297 <Peterwayne3293@gmail.com>
Date:   Tue Apr 2 15:00:35 2024 -0400

    cleanup odrive GUI related code

commit 56246f7684a0f9716a773e23200e05410f66f2d7
Author: mn297 <Peterwayne3293@gmail.com>
Date:   Tue Apr 2 12:39:14 2024 -0400

    launch file for drive

commit d0953d8ac4f158c3e19794a9448996d767d0018a
Author: mn297 <Peterwayne3293@gmail.com>
Date:   Mon Apr 1 19:08:52 2024 -0400

    drive gui

commit 560b2813e46b84a248f477ee2f252da141eecb11
Author: mn297 <Peterwayne3293@gmail.com>
Date:   Mon Apr 1 18:31:41 2024 -0400

    fixed drive simultaneous config

commit a230b61633439214bb09c61a9040bb0e1e7f7873
Author: mn297 <Peterwayne3293@gmail.com>
Date:   Mon Apr 1 15:36:50 2024 -0400

    debugging drive

commit 31f971173c36780fea81563619a86acfd5566cea
Author: mn297 <Peterwayne3293@gmail.com>
Date:   Mon Apr 1 01:46:21 2024 -0400

    changed drive_control

commit b0766d22816d3ec2dea2c815871851fc3f28b9f2
Author: mn297 <Peterwayne3293@gmail.com>
Date:   Sun Mar 31 23:16:21 2024 -0400

    fixed typo

commit af16e5680824b8b6f8ff7a1d388abef64c6da790
Author: Your Name <peterwayne3293@gmail.com>
Date:   Sun Mar 31 18:54:18 2024 -0400

    fixed arm naming

commit eff2291f6527bd1884cd0c4dccfaa87150d8f26e
Author: Your Name <peterwayne3293@gmail.com>
Date:   Sun Mar 31 18:40:05 2024 -0400

    initial drive odrive interface

commit 95302049c27463096e62d38a9002562cd1f5e43a
Author: mn297 <Peterwayne3293@gmail.com>
Date:   Sat Mar 30 23:00:13 2024 -0400

    reorganized packages

commit 7727f87b28dc2a07cefefa2ddf3b67b8323df0b3
Author: mn297 <Peterwayne3293@gmail.com>
Date:   Sat Mar 30 21:52:18 2024 -0400

    renamed joints to standard

commit ba7f210a744e9ee90c8c7ea890839bdcc19ade35
Author: Your Name <peterwayne3293@gmail.com>
Date:   Mon Mar 18 19:43:10 2024 -0400

    limswitch config

commit b6122a96e22cb501f651b99eb97a093e4c1045bb
Author: Your Name <peterwayne3293@gmail.com>
Date:   Mon Mar 18 19:38:53 2024 -0400

    tester script cleanup

commit 06e17f5f243063033c122fc8dc0d7119187f532f
Author: Your Name <peterwayne3293@gmail.com>
Date:   Mon Mar 18 19:37:14 2024 -0400

    variable names

commit 8c5a44a1303f994d9021aa24fe881bc01a1da447
Author: Your Name <peterwayne3293@gmail.com>
Date:   Sun Mar 17 18:53:38 2024 -0400

    cleanup

commit 2f4b588d936adf6867e29938c2eeb6ac2915b75a
Author: mn297 <Peterwayne3293@gmail.com>
Date:   Sun Mar 17 14:36:02 2024 -0400

    fixed typo topic name

commit 6eb678c21ce86b0f2507ec5bc6504dfe8e6ab082
Author: mn297 <Peterwayne3293@gmail.com>
Date:   Sun Mar 17 01:33:46 2024 -0400

    vel_limit

commit 9c774e71f480600049b69f9ac2b9fba70a6e5034
Author: mn297 <Peterwayne3293@gmail.com>
Date:   Sat Mar 16 23:50:46 2024 -0400

    gui tester done

commit d7eb3287b1399f8145d244bedb64433e94141cbe
Author: mn297 <Peterwayne3293@gmail.com>
Date:   Sat Mar 16 23:38:05 2024 -0400

    gui tester

commit 112db609f36caa09da1dfc1e7b24c30c89b28299
Author: mn297 <Peterwayne3293@gmail.com>
Date:   Sat Mar 16 22:39:26 2024 -0400

    2 motors working

commit 202d892dd5cdde7e73760f5de9e2f8d660fbf961
Author: mn297 <Peterwayne3293@gmail.com>
Date:   Sat Mar 16 19:28:46 2024 -0400

    fixed typo serial

commit bd5c779fac974d3eb5cd20376d8e6f22a004d80d
Author: mn297 <Peterwayne3293@gmail.com>
Date:   Sat Mar 16 12:29:58 2024 -0400

    elbow serial

commit 4c76860ac30e0c2a999c4fd389f23dc43f40a7fe
Author: Your Name <peterwayne3293@gmail.com>
Date:   Sat Mar 16 01:52:06 2024 -0400

    added comments

commit f5669f7568dbf11412e69d0b34c76f134c3bc9ed
Author: Your Name <peterwayne3293@gmail.com>
Date:   Thu Feb 1 13:59:48 2024 -0500

    added package for odrive arm

File: arm_control/model/MR_arm.urdf (robot description, URDF)
Before this commit: robot mr_arm, 8 links, 7 joints
Links:
- link link_0: geometry collision mesh filename=package://arm_control/model/meshes/collision_Link0.stl; visual mesh filename=package://arm_control/model/meshes/Link0.stl
- link link_1: geometry collision mesh filename=package://arm_control/model/meshes/collision_Link1.stl; visual mesh filename=package://arm_control/model/meshes/Link1.stl
- link link_2: geometry collision mesh filename=package://arm_control/model/meshes/collision_Link2.stl; visual mesh filename=package://arm_control/model/meshes/Link2.stl
- link link_3: geometry collision mesh filename=package://arm_control/model/meshes/collision_Link3.stl; visual mesh filename=package://arm_control/model/meshes/Link3.stl
- link link_4: geometry collision mesh filename=package://arm_control/model/meshes/collision_Link4.stl; visual mesh filename=package://arm_control/model/meshes/Link4.stl
- link link_5: geometry collision mesh filename=package://arm_control/model/meshes/collision_Link5.stl; visual mesh filename=package://arm_control/model/meshes/Link5.stl
- link link_6: geometry collision box size=0.1 0.1 0.1; visual mesh filename=package://arm_control/model/meshes/finger.stl
- link link_7: geometry collision box size=0.1 0.1 0.1; visual mesh filename=package://arm_control/model/meshes/finger.stl
Joints:
- removed joint joint_1
- removed joint joint_2
- removed joint joint_3
- removed joint joint_4
- removed joint joint_5
- removed joint joint_6
- added joint joint_elbow: type revolute, parent link_2, child link_3, origin xyz=0 0 0.5 rpy=0 0 0, axis 0 1 0, limit lower=-1.570796327 upper=1.570796327 effort=10.0 velocity=2.61799
- added joint joint_end_effector: type revolute, parent link_5, child link_6, origin xyz=0.050 -0.045 -0.01 rpy=0 0 1.570796327, axis 0 0 1, limit lower=-3.141592 upper=3.141592 effort=10.0 velocity=2.61799
- added joint joint_shoulder: type revolute, parent link_1, child link_2, origin xyz=0 0 0.0575 rpy=0 0 0, axis 0 1 0, limit lower=-1.570796327 upper=1.570796327 effort=10.0 velocity=2.61799
- added joint joint_waist: type revolute, parent link_0, child link_1, origin xyz=0 0 0 rpy=0 0 0, axis 0 0 1, limit lower=-3.141592 upper=3.141592 effort=10.0 velocity=2.61799
- added joint joint_wrist_pitch: type revolute, parent link_3, child link_4, origin xyz=0.4 0 0 rpy=0 0 0, axis 0 1 0, limit lower=-1.570796327 upper=1.570796327 effort=10.0 velocity=2.61799
- added joint joint_wrist_roll: type revolute, parent link_4, child link_5, origin xyz=0.034 0 0 rpy=0 0 0, axis 1 0 0, limit lower=-3.141592 upper=3.141592 effort=10.0 velocity=2.61799
